Commit message: Put the arms on the real HIL table: hanging chaser, debris on tabletop
Layout (CAD values from HIL_Main_Robotics):
- Chaser arm hangs upside-down from the overhead MISUMI E-MTHE17 rail
  carriage (rail frame Rx(pi), carriage at stroke 0 = x -0.795, mount
  face z 0.773). Stroke 0 assumed at the -X (drawer-box) end.
- Debris arm stands on the 1.39 x 0.74 m tabletop at (0.55, -0.29, 0),
  holding the target at (0.64, 0, 0.35).
- Satellite height 0.35 m (at 0.30 the debris arm has no level pose
  from a base on the table).
- Approach trimmed to start at 1.30 m range (the rail stroke can't
  cover 1.5 m with the target on the table); the CSV is unchanged.
- Standoff 0.23 m ahead of the carriage, ramping smoothly from 0.13 m
  over the first 150 s so the arm doesn't swing at the start.
- Chaser mock-up mounted 180 deg about the tool axis (joint 6 would
  otherwise need +/-pi, outside its limit).

Script: multi-start IK, frame/table/rail checks, IK acceptance line,
eased moves into the start and test poses (no step changes sent to
Unity or the hardware bridge). IK: 0.007 mm / 0.03 deg, joints >= 0.067
rad from limits.

Unity: imported HIL table/frame/rail FBX with CAD materials, robots
placed, CAD carriage parented to rail_carriage on Play, URDF rail boxes
hidden, Run In Background on.

File: UnityProject/Assets/RS/ReBot_Chaser_Rail.urdf (robot description, URDF)
Before this commit: robot ReBot_Chaser_Rail, 12 links, 11 joints
Links:
- link rail_base: geometry 
- link rail_carriage: geometry visual box size=0.14 0.14 0.02
